File: pcb/ESPHome-Parking-Assistant.kicad_pcb (KiCad board)
At the start: 4 copper layers, 85 x 59 mm, 114 parts, among them J1 TYPE-C-31-M-12, J2 533980471, J3 533980671, J4 Screw_Terminal_01x04, Q1 STL9P3LLH6, SW1 RESET, SW2 BOOT, U1 STUSB4500, U2 INA228, U3 TPS560430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

Commit message: Change R23 to 15KΩ
Parts:
- R23: value 22KΩ -> 15KΩ
- R26: value 15KΩ -> DNP
