File: pcb/esp32.kicad_sch (KiCad schematic)
At the start: 31 parts, among them J2 533980471, J3 533980671, J4 Screw_Terminal_01x04, SW1 RESET, SW2 BOOT, U5 ESP32-S3-WROOM-1, U6 TC4427, U7 SN74LV1T34DBV

Commit message: Fix last commit. R26 is DNP and R23 changed to 15kΩ.
Parts:
- R31, R32, R33, R34, R35, R36: Comment Resistor -> (none)
Changed lines of the file:
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@@
 			)
 		)
-		(property "Comment" "Resistor"
+		(property "Comment" ""
 			(at 172.72 102.87 0)
 			(effects
@@
 			)
 		)
-		(property "Comment" "Resistor"
+		(property "Comment" ""
 			(at 99.06 44.45 0)
 			(effects
@@
 			)
 		)
-		(property "Comment" "Resistor"
+		(property "Comment" ""
 			(at 162.56 44.45 0)
 			(effects
@@
 			)
 		)
-		(property "Comment" "Resistor"
+		(property "Comment" ""
 			(at 182.88 44.45 0)
 			(effects
@@
 			)
 		)
-		(property "Comment" "Resistor"
+		(property "Comment" ""
 			(at 172.72 44.45 0)
 			(effects
@@
 			)
 		)
-		(property "Comment" "Resistor"
+		(property "Comment" ""
 			(at 109.22 44.45 0)
 			(effects
