File: pcb/Power-Supplies.kicad_sch (KiCad schematic)
At the start: 47 parts, among them U3 TPS560430, U4 TPS552872RYQR

Commit message: Update to KiCad  10.0.6 No functional changes to design
Parts:
- NT1: value ~ -> (none)
